File: ino5x6/ino5x6.sch (KiCad schematic (older format))
At the start: 74 parts, among them J1 Conn_01x04_Male, J2 Conn_01x01_Male, J3 Conn_01x01_Male, J4 Conn_01x01_Male, J5 Conn_01x01_Male, SW1 SW_Push, SW10 SW_Push, SW11 SW_Push, SW12 SW_Push, SW13 SW_Push, SW14 SW_Push, SW15 SW_Push, SW16 SW_Push, SW17 SW_Push, SW18 SW_Push, SW19 SW_Push, SW2 SW_Push, SW20 SW_Push, SW21 SW_Push, SW22 SW_Push, SW23 SW_Push, SW24 SW_Push, SW25 SW_Push, SW26 SW_Push, SW27 SW_Push, SW28 SW_Push, SW29 SW_Push, SW3 SW_Push, SW30 SW_Push, SW4 SW_Push, SW5 SW_Push, SW6 SW_Push, SW7 SW_Push, SW8 SW_Push, SW9 SW_Push, U1 ProMicro

Commit message: 配置の厳密化
Parts:
- added MH1, MH2, MH3, MH4: MountingHole, Mounting_Holes:MountingHole_3.2mm_M3, symbol Mechanical:MountingHole
Changed lines of the file:
@@
 	1800 3000 1500 3000
 Wire Wire Line
-	1800 2900 1500 2900
-Text Label 1500 2900 0    50   ~ 0
+	1800 2800 1500 2800
+Text Label 1500 2800 0    50   ~ 0
 row0
 Text Label 1500 3000 0    50   ~ 0
@@
 NoConn ~ 3200 2200
 NoConn ~ 3200 2600
-NoConn ~ 1800 2800
 NoConn ~ 1800 2300
 NoConn ~ 3200 2700
@@
 	0    1    1    0
 $EndComp
+NoConn ~ 1800 2900
+$Comp
+L Mechanical:MountingHole MH2
+U 1 1 5B9FB144
+P 1700 6450
+F 0 "MH2" H 1800 6496 50  0000 L CNN
+F 1 "MountingHole" H 1800 6405 50  0000 L CNN
+F 2 "Mounting_Holes:MountingHole_3.2mm_M3" H 1700 6450 50  0001 C CNN
+F 3 "~" H 1700 6450 50  0001 C CNN
+	1    1700 6450
+	1    0    0    -1
+$EndComp
+$Comp
+L Mechanical:MountingHole MH1
+U 1 1 5B9FB28E
+P 1700 6200
+F 0 "MH1" H 1800 6246 50  0000 L CNN
+F 1 "MountingHole" H 1800 6155 50  0000 L CNN
+F 2 "Mounting_Holes:MountingHole_3.2mm_M3" H 1700 6200 50  0001 C CNN
+F 3 "~" H 1700 6200 50  0001 C CNN
+	1    1700 6200
+	1    0    0    -1
+$EndComp
+$Comp
+L Mechanical:MountingHole MH3
+U 1 1 5B9FB478
+P 1700 6700
+F 0 "MH3" H 1800 6746 50  0000 L CNN
+F 1 "MountingHole" H 1800 6655 50  0000 L CNN
+F 2 "Mounting_Holes:MountingHole_3.2mm_M3" H 1700 6700 50  0001 C CNN
+F 3 "~" H 1700 6700 50  0001 C CNN
+	1    1700 6700
+	1    0    0    -1
+$EndComp
+$Comp
+L Mechanical:MountingHole MH4
+U 1 1 5B9FB53A
+P 1700 6950
+F 0 "MH4" H 1800 6996 50  0000 L CNN
+F 1 "MountingHole" H 1800 6905 50  0000 L CNN
+F 2 "Mounting_Holes:MountingHole_3.2mm_M3" H 1700 6950 50  0001 C CNN
+F 3 "~" H 1700 6950 50  0001 C CNN
+	1    1700 6950
+	1    0    0    -1
+$EndComp
 $EndSCHEMATC

Commit message: クリアランスと太さを0.3に
Parts:
- JP1, JP2, JP3, JP4: footprint Pin_Headers:Pin_Header_Straight_1x02_Pitch2.54mm -> Wire_Connections_Bridges:WireConnection_0.80mmDrill
Changed lines of the file:
@@
 F 0 "JP1" V 6054 2358 50  0000 L CNN
 F 1 "Jumper_2_Bridged" V 6150 1800 50  0000 L CNN
-F 2 "Pin_Headers:Pin_Header_Straight_1x02_Pitch2.54mm" H 6100 2300 50  0001 C CNN
+F 2 "Wire_Connections_Bridges:WireConnection_0.80mmDrill" H 6100 2300 50  0001 C CNN
 F 3 "~" H 6100 2300 50  0001 C CNN
 	1    6100 2300
@@
 F 0 "JP2" V 6954 3158 50  0000 L CNN
 F 1 "Jumper_2_Bridged" V 7050 2600 50  0000 L CNN
-F 2 "Pin_Headers:Pin_Header_Straight_1x02_Pitch2.54mm" H 7000 3100 50  0001 C CNN
+F 2 "Wire_Connections_Bridges:WireConnection_0.80mmDrill" H 7000 3100 50  0001 C CNN
 F 3 "~" H 7000 3100 50  0001 C CNN
 	1    7000 3100
@@
 F 0 "JP3" V 7854 3958 50  0000 L CNN
 F 1 "Jumper_2_Bridged" V 7950 3400 50  0000 L CNN
-F 2 "Pin_Headers:Pin_Header_Straight_1x02_Pitch2.54mm" H 7900 3900 50  0001 C CNN
+F 2 "Wire_Connections_Bridges:WireConnection_0.80mmDrill" H 7900 3900 50  0001 C CNN
 F 3 "~" H 7900 3900 50  0001 C CNN
 	1    7900 3900
@@
 F 0 "JP4" V 8754 4758 50  0000 L CNN
 F 1 "Jumper_2_Bridged" V 8850 4200 50  0000 L CNN
-F 2 "Pin_Headers:Pin_Header_Straight_1x02_Pitch2.54mm" H 8800 4700 50  0001 C CNN
+F 2 "Wire_Connections_Bridges:WireConnection_0.80mmDrill" H 8800 4700 50  0001 C CNN
 F 3 "~" H 8800 4700 50  0001 C CNN
 	1    8800 4700
